File: kicad/Breadbord-pc/Breadbord-pc.kicad_sch (KiCad schematic)
At the start: 14 parts, among them SW1 SW_Push, U1 8088, U11 8255A, U2 74HC573, U3 74HC573, U4 W29C020C, U6 74HC245, U7 74HC573, U8 HM628128D, U9 74HCT00

Commit message: Mise en place du schéma
Parts:
- IC-6, U9: footprint (none) -> Package_DIP:DIP-14_W7.62mm
- U3, U6: footprint (none) -> Package_DIP:DIP-20_W7.62mm
Other:
- company: By VE2CUY -> (none)
- title: 8088 - Breadboard -> (none)
