File: kicad/Breadboard-pc/Breadboard-pc.kicad_sch (KiCad schematic)
At the start: 14 parts, among them SW1 SW_Push, U1 8088, U11 8255A, U2 74HC573, U3 74HC573, U4 W29C020C, U6 74HC245, U7 74HC573, U8 HM628128D, U9 74HCT00

Commit message: Actualisé le PCB
Parts:
- removed BAR1: HDSP-4850_2, Display:HDSP-4850, symbol LED:HDSP-4850_2
- removed RN1: R_333 Network, Resistor_THT:R_Array_SIP10, symbol Device:R_Network09
- removed U7: 74HC573, Package_DIP:DIP-20_W7.62mm, symbol 74xx:74LS573
- added D1: PWR, LED_THT:LED_D3.0mm, symbol Device:LED
- added J1: USB_A (clavier PS/2), Connector_USB:USB_A_Molex_67643_Horizontal, symbol Connector:USB_A
- added J2: LCD I2C, Connector_PinHeader_2.54mm:PinHeader_1x04_P2.54mm_Vertical, symbol Connector:Conn_01x04_Pin
- added J3: 5V 2A, Connector_BarrelJack:BarrelJack_Horizontal, symbol Connector:Barrel_Jack
- added J4: CLK externe, Connector_PinHeader_2.54mm:PinHeader_1x02_P2.54mm_Vertical, symbol Connector:Conn_01x02_Pin
- added JP1: 1-2: STM32 2-3: ext., Connector_PinHeader_2.54mm:PinHeader_1x03_P2.54mm_Vertical, symbol Jumper:Jumper_3_Open
- added R2, R3, R4, R7: 10k, Resistor_THT:R_Axial_DIN0207_L6.3mm_D2.5mm_P7.62mm_Horizontal, symbol Device:R_Small_US
- added R5, R6: 4.7k, Resistor_THT:R_Axial_DIN0207_L6.3mm_D2.5mm_P7.62mm_Horizontal, symbol Device:R_Small_US
- added R8: 1k, Resistor_THT:R_Axial_DIN0207_L6.3mm_D2.5mm_P7.62mm_Horizontal, symbol Device:R_Small_US
- added SW2: IR0 test, Button_Switch_THT:SW_PUSH_6mm, symbol Switch:SW_Push
- added U5: STM32F411 BlackPill, WeAct_Black_Pill_V2.0:STM32F411_Black_Pill, symbol Bread-board-PC:STM32F411_Black_Pill_VE2CUY
- added U7: 8259A, Package_DIP:DIP-28_W15.24mm, symbol Interface:8259A
- added unit 2 of U9
- added unit 5 of U9
- R1: footprint (none) -> Resistor_THT:R_Axial_DIN0207_L6.3mm_D2.5mm_P7.62mm_Horizontal
- SW1: value SW_Push -> RESET; footprint (none) -> Button_Switch_THT:SW_PUSH_6mm
- U2: value 74HC573 -> 74LS373; footprint (none) -> Package_DIP:DIP-20_W7.62mm; symbol 74xx:74LS573 -> 74xx:74LS373
- U3: value 74HC573 -> 74LS373; symbol 74xx:74LS573 -> 74xx:74LS373
- U4: footprint Package_DIP:DIP-32_W15.24mm -> Socket:DIP_Socket-32_W11.9mm_W12.7mm_W15.24mm_W17.78mm_W18.5mm_3M_232-1285-00-0602J
- U9: value 74HCT00 -> 74LS00; symbol 74xx:74HCT00 -> 74xx:74LS00
Connections:
- net +5V: now also J1.1 (VBUS), J2.2 (Pin_2), J3.1, R2.1, R3.1, R5.1, R6.1, R8.1, SW2.2, U5.18 (5V), U5.40 (5V), U7.16 (~{SP}/~{EN}), U7.28 (VCC), U9.14 (VCC)
- net A0: now also U2.2 (O0), U7.27 (A0); no longer U2.19 (Q0)
- net A1: now also U2.5 (O1); no longer U2.18 (Q1)
- net A12: now also U3.2 (O0); no longer U3.19 (Q0)
- net A13: now also U3.5 (O1); no longer U3.18 (Q1)
- net A14: now also U3.6 (O2); no longer U3.17 (Q2)
- net A15: now also U3.9 (O3); no longer U3.16 (Q3)
- net A16: now also U3.12 (O4); no longer U3.15 (Q4)
- net A17: now also U3.15 (O5); no longer U3.14 (Q5)
- net A18: now also U3.16 (O6); no longer U3.13 (Q6)
- net A19: now also U3.19 (O7); no longer U3.12 (Q7)
- net A2: now also U2.6 (O2); no longer U2.17 (Q2)
- net A3: now also U2.9 (O3); no longer U2.16 (Q3)
- net A4: now also U2.12 (O4); no longer U2.15 (Q4)
- net A5: now also U2.15 (O5), U9.5; no longer U2.14 (Q5)
- net A6: now also U2.16 (O6); no longer U2.13 (Q6)
- net A7: now also U2.19 (O7); no longer U2.12 (Q7)
- net D0: now also U7.11 (D0)
- net D1: now also U7.10 (D1)
- net D2: now also U7.9 (D2)
- net D3: now also U7.8 (D3)
- net D4: now also U7.7 (D4)
- net D5: now also U7.6 (D5)
- net D6: now also U7.5 (D6)
- net D7: now also U7.4 (D7)
- net GND: now also D1.1 (K), J1.4 (GND), J1.SH (Shield), J2.1 (Pin_1), J3.2, J4.2 (Pin_2), R4.2, R7.2, U5.19 (G), U5.39 (G), U7.14 (GND), U7.20 (IR2), U7.21 (IR3), U7.22 (IR4), U7.23 (IR5), U7.24 (IR6), U7.25 (IR7), U9.7 (GND); no longer U1.18 (INTR)
- net RD_: now also U7.3 (~{RD})
- net RESET: now also U5.36 (B2)
- net WR_: now also U7.2 (~{WR})
- net IO: now reaches IC-6.1, IC-6.2, U1.28 (IO/~{M}), U9.1
- net IO: now also U9.4
- net at U1.10 (AD6), U6.8 (A6): now also U2.17 (D6); no longer U2.8 (D6)
- net at U1.11 (AD5), U6.7 (A5): now also U2.14 (D5); no longer U2.7 (D5)
- net at U1.12 (AD4), U6.6 (A4): now also U2.13 (D4); no longer U2.6 (D4)
- net at U1.13 (AD3), U6.5 (A3): now also U2.8 (D3); no longer U2.5 (D3)
- net at U1.14 (AD2), U6.4 (A2): now also U2.7 (D2); no longer U2.4 (D2)
- net at U1.15 (AD1), U6.3 (A1): now also U2.4 (D1); no longer U2.3 (D1)
- net at U1.16 (AD0), U6.2 (A0): now also U2.3 (D0); no longer U2.2 (D0)
- net CLK: now reaches U1.19 (CLK)
- net CLK: now also JP1.2 (C)
- net at U1.2 (A14): now also U3.7 (D2); no longer U3.4 (D2)
- net INTA_: now reaches U1.24 (~{INTA})
- net INTA_: now also U7.26 (~{INTA})
- net at U1.3 (A13): now also U3.4 (D1); no longer U3.3 (D1)
- net at U1.35 (A19/S6): now also U3.18 (D7); no longer U3.9 (D7)
- net at U1.36 (A18/S5): now also U3.17 (D6); no longer U3.8 (D6)
- net at U1.37 (A17/S4): now also U3.14 (D5); no longer U3.7 (D5)
- net at U1.38 (A16/S3): now also U3.13 (D4); no longer U3.6 (D4)
- net at U1.39 (A15): now also U3.8 (D3); no longer U3.5 (D3)
- net at U1.4 (A12): now also U3.3 (D0); no longer U3.2 (D0)
- net at U1.9 (AD7), U6.9 (A7): now also U2.18 (D7); no longer U2.9 (D7)
- net BUS_PA3: now reaches U11.1 (PA3)
- net BUS_PA3: now also U5.4 (B15)
- net OBF_: now reaches U11.10 (PC7)
- net OBF_: now also U5.5 (A8)
- net ACK_: now reaches U11.11 (PC6)
- net ACK_: now also R2.2, U5.34 (B0)
- net IBF: now reaches U11.12 (PC5)
- net IBF: now also U5.10 (A15)
- net STB_: now reaches U11.13 (PC4)
- net STB_: now also R3.2, U5.35 (B1)
- net TAG: now reaches U11.14 (PC0)
- net TAG: now also U5.12 (B4)
- net TAG1: now reaches U11.15 (PC1)
- net TAG1: now also R4.1, U5.13 (B5)
- net IRQ1: now reaches U11.17 (PC3)
- net IRQ1: now also U7.19 (IR1)
- net CANAL0: now reaches U11.18 (PB0)
- net CANAL0: now also U5.6 (A9)
- net CANAL1: now reaches U11.19 (PB1)
- net CANAL1: now also U5.7 (A10)
- net BUS_PA2: now reaches U11.2 (PA2)
- net BUS_PA2: now also U5.3 (B14)
- net BUS_PA1: now reaches U11.3 (PA1)
- net BUS_PA1: now also U5.2 (B13)
- net BUS_PA7: now reaches U11.37 (PA7)
- net BUS_PA7: now also U5.14 (B6)
- net BUS_PA6: now reaches U11.38 (PA6)
- net BUS_PA6: now also U5.15 (B7)
- net BUS_PA5: now reaches U11.39 (PA5)
- net BUS_PA5: now also U5.16 (B8)
- net BUS_PA0: now reaches U11.4 (PA0)
- net BUS_PA0: now also U5.1 (B12)
- net BUS_PA4: now reaches U11.40 (PA4)
- net BUS_PA4: now also U5.17 (B9)
- new net: R7.1, SW2.1, U7.18 (IR0)
- new net: D1.2 (A), R8.2
- new net CLK_EXT: J4.1 (Pin_1), JP1.3 (B)
- new net CLK_STM: JP1.1 (A), U5.29 (A3)
- new net CS8259_: U7.1 (~{CS}), U9.6
- new net INTR: U1.18 (INTR), U7.17 (INT)
- new net LCD_SCL: J2.4 (Pin_4), U5.37 (B10)
- new net LCD_SDA: J2.3 (Pin_3), U5.11 (B3)
- new net PS2_CLK: J1.3 (D+), R5.2, U5.27 (A1)
- new net PS2_DATA: J1.2 (D-), R6.2, U5.28 (A2)
- no-connect marks 26 -> 28
Other:
- added sheet STM32 Bridge (untitled.kicad_sch)
- note added: "0000h-1FFFFh"
- note added: "8088 on Breadboard - Version 1.0"
- note added: "C0000h-FFFFFh"
- note removed: "* IO OUT on any port will trigger latch"
- note removed: "<-- RAM Select: 0000h-1FFFFh"
- note removed: "<-- ROM Select : C0000h-FFFFFh"
- note removed: "D0"
- note removed: "D1"
- note removed: "D2"
- note removed: "D3"
- note removed: "D4"
- note removed: "D5"
- note removed: "D6"
- note removed: "D7"
- note removed: "IC-08"
- moved on the sheet: IC-6A, IC-6B, IC-6C, IC-6D, IC-6E, R1, SW1, U11
